File: voltage_measure_pcb.sch (KiCad schematic (older format))
At the start: 10 parts, among them J1 Conn_01x03_Male, J2 Conn_01x02_Male, Q1 BSS84, Q2 BSS123

Commit message: missing EN wire fixed
Connections:
- net EN: now also J1.1 (Pin_1)
Changed lines of the file:
@@
 Wire Wire Line
 	6500 3850 6500 4350
+Wire Wire Line
+	3850 2900 4300 2900
 $EndSCHEMATC
